Commit message: first

File: exp6_urdf_demo/urdf/urdf/base_footprint_urdf.urdf (robot description, URDF)
Before this commit: robot car, 2 links, 1 joints
Links:
- added link base_footprint; visual box size=0.0001 0.0001 0.001
- link base_link: geometry visual box size=0.4 0.3 0.1
Joints:
- added joint base_footprint2base: type fixed, parent base_footprint, child base_link, origin xyz=0.0 0 0.05 rpy=0 0 0
